File: ETI vocoder/internal excitation- #7.sch (EAGLE design)
At the start: 51 parts, among them IC1 LM1458N, IC3 TL081P, IC4 UA741P, IC5 4006N, IC6 4030N, IC7 LM1458N, Q1 BC182L

Commit message: Fixed input boards in regards to article and added spacer holes
Parts:
- removed BOARD1: 22-23-2041, con-molex:22-23-2041
- removed BOARD1-PWR: 22-23-2021, con-molex:22-23-2021
- removed R18: 47k, resistor:R-EU_0207/7
- added CARD2: (no value), con-molex:22-23-2061
- C1, C8: device resistor:C-EU075-032X103 -> resistor:C-EU050-025X075
- C2: value 10n -> 100n
- C6: value 33n -> 100n; device resistor:C-EU075-032X103 -> resistor:C-EU025-025X050
- R10: value 3k3 -> 1k
- renumbered C9 to C3, R49 to R10
Connections:
- removed net N$22: R18.2, RV7G$1.1S
- net BOARD2_MIX: now also CARD2-4.S, RV7G$1.1S; no longer BOARD1-4.S, R18.1
- net GND: now also RV5G$1.1A, RV7G$1.1E; no longer IC5P.VSS, IC6P.VSS, RV5G$1.1E, RV7G$1.1A
- net N$15: now also D1.A, D2.C; no longer D1.C, D2.A
- net N$17: now also D1.C; no longer D2.C
- net N$18: now also D2.A; no longer D1.A
- net N$9: now also RV5G$1.1E; no longer RV5G$1.1A
- net VCA_CTRL: now also CARD2-2.S; no longer BOARD1-2.S
- net VCA_SIGNAL: now also CARD2-1.S, RV7G$1.1A; no longer BOARD1-3.S, RV7G$1.1E
- net VDD: now also CARD2-5.S; no longer BOARD1-PWR-2.S
- net VSS: now also CARD2-6.S, IC5P.VSS, IC6P.VSS; no longer BOARD1-PWR-1.S
- net X: now also CARD2-3.S; no longer BOARD1-1.S
Other:
- note added: "NB: IC5 and IC6 are mixed up in the original datasheet"
- note added: "Sjekk retning på pots!"
- note removed: "NB: IC5 and IC6 are mixed in the original datasheet vs parts list. This follows the parts list"
- note removed: "R18 is missing from the article"
- note removed: "Sjekket caps og pots"
- note removed: "Sjekket opp mot artikkel og board"
- moved on the sheet: D1, D2, RV5, RV7
