File: ETI vocoder/led ppm display.sch (EAGLE design)
At the start: 29 parts, among them IC1 TL082P, IC2 LM3915N

Commit message: Fixed input boards in regards to article and added spacer holes
Other:
- note added: "Sjekket caps ok"
Changed lines of the file:
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@@
 <?xml version="1.0" encoding="utf-8"?>
 <!DOCTYPE eagle SYSTEM "eagle.dtd">
-<eagle version="7.2.0">
+<eagle version="6.2">
 <drawing>
 <settings>
@@
 <text x="187.96" y="25.4" size="1.778" layer="97" rot="R90">Red</text>
 <text x="187.96" y="50.8" size="1.778" layer="97" rot="R90">Green</text>
+<text x="43.18" y="78.74" size="1.778" layer="91">Sjekket caps ok</text>
 </plain>
 <instances>
@@
 </schematic>
 </drawing>
-<compatibility>
-<note version="6.3" minversion="6.2.2" severity="warning">
-Since Version 6.2.2 text objects can contain more than one line,
-which will not be processed correctly with this version.
-</note>
-</compatibility>
 </eagle>

Commit message: Finished first of two halves of the universal voice board
Connections:
- removed net N$10: IC2.REFADJ, R7.2
- new net N$21: IC2.REFADJ, R7.1, R8.2
- net N$1: now also D1.A; no longer D2.A
- net N$2: now also D2.C; no longer D1.C
- net N$3: now also D1.C, D2.A; no longer D1.A, D2.C
- net N$4: now also D4.A; no longer D3.A
- net N$5: now also D3.C; no longer D4.C
- net N$7: now also D3.A, D4.C; no longer D3.C, D4.A
- net N$9: now also R7.2; no longer R7.1, R8.2
Other:
- note added: "R7 is misplaced in the schematics in the original article"
- note removed: "Sjekket caps ok"
- moved on the sheet: D1, D2, D3, D4, R7
Changed lines of the file:
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@@
 <parts>
 <part name="IC1" library="linear" deviceset="TL082" device="P"/>
+<part name="D2" library="joakim" deviceset="1N4148" device="DOJ35-5" value="1N4148DOJ35-5"/>
 <part name="D1" library="joakim" deviceset="1N4148" device="DOJ35-5" value="1N4148DOJ35-5"/>
-<part name="D2" library="joakim" deviceset="1N4148" device="DOJ35-5" value="1N4148DOJ35-5"/>
+<part name="D4" library="joakim" deviceset="1N4148" device="DOJ35-5" value="1N4148DOJ35-5"/>
 <part name="D3" library="joakim" deviceset="1N4148" device="DOJ35-5" value="1N4148DOJ35-5"/>
-<part name="D4" library="joakim" deviceset="1N4148" device="DOJ35-5" value="1N4148DOJ35-5"/>
 <part name="R1" library="resistor" deviceset="R-EU_" device="0207/7" value="100k"/>
 <part name="R2" library="resistor" deviceset="R-EU_" device="0207/7" value="100k"/>
@@
 <text x="187.96" y="25.4" size="1.778" layer="97" rot="R90">Red</text>
 <text x="187.96" y="50.8" size="1.778" layer="97" rot="R90">Green</text>
-<text x="43.18" y="78.74" size="1.778" layer="91">Sjekket caps ok</text>
+<text x="106.68" y="81.28" size="1.778" layer="97">R7 is misplaced in the schematics in the original article</text>
 </plain>
 <instances>
@@
 </instance>
 <instance part="IC1" gate="P" x="83.82" y="0"/>
-<instance part="D1" gate="G$1" x="76.2" y="43.18" smashed="yes" rot="R180">
+<instance part="D2" gate="G$1" x="76.2" y="43.18" smashed="yes" rot="R180">
 <attribute name="NAME" x="73.66" y="42.6974" size="1.778" layer="95" rot="R180"/>
 </instance>
-<instance part="D2" gate="G$1" x="76.2" y="48.26" smashed="yes">
+<instance part="D1" gate="G$1" x="76.2" y="48.26" smashed="yes">
 <attribute name="NAME" x="78.74" y="48.7426" size="1.778" layer="95"/>
 </instance>
-<instance part="D3" gate="G$1" x="101.6" y="63.5" smashed="yes">
+<instance part="D4" gate="G$1" x="101.6" y="63.5" smashed="yes">
 <attribute name="NAME" x="104.14" y="63.9826" size="1.778" layer="95"/>
 </instance>
-<instance part="D4" gate="G$1" x="101.6" y="68.58" smashed="yes" rot="R180">
+<instance part="D3" gate="G$1" x="101.6" y="68.58" smashed="yes" rot="R180">
 <attribute name="NAME" x="104.14" y="69.0626" size="1.778" layer="95"/>
 </instance>
@@
 <attribute name="VALUE" x="116.078" y="67.31" size="1.778" layer="96" rot="R270"/>
 </instance>
-<instance part="R7" gate="G$1" x="134.62" y="50.8"/>
+<instance part="R7" gate="G$1" x="121.92" y="55.88" rot="R90"/>
 <instance part="R8" gate="G$1" x="121.92" y="45.72" rot="R90"/>
 <instance part="GND1" gate="1" x="88.9" y="43.18"/>
@@
 <segment>
 <pinref part="R2" gate="G$1" pin="1"/>
-<pinref part="D2" gate="G$1" pin="A"/>
+<pinref part="D1" gate="G$1" pin="A"/>
 <wire x1="71.12" y1="48.26" x2="73.66" y2="48.26" width="0.1524" layer="91"/>
 <wire x1="73.66" y1="48.26" x2="73.66" y2="55.88" width="0.1524" layer="91"/>
@@
 <net name="N$2" class="0">
 <segment>
-<pinref part="D1" gate="G$1" pin="C"/>
+<pinref part="D2" gate="G$1" pin="C"/>
 <wire x1="73.66" y1="43.18" x2="60.96" y2="43.18" width="0.1524" layer="91"/>
 <wire x1="60.96" y1="43.18" x2="60.96" y2="35.56" width="0.1524" layer="91"/>
@@
 <net name="N$3" class="0">
 <segment>
-<pinref part="D2" gate="G$1" pin="C"/>
+<pinref part="D1" gate="G$1" pin="C"/>
 <wire x1="78.74" y1="48.26" x2="81.28" y2="48.26" width="0.1524" layer="91"/>
 <wire x1="81.28" y1="48.26" x2="81.28" y2="43.18" width="0.1524" layer="91"/>
@@
 <wire x1="81.28" y1="43.18" x2="81.28" y2="33.02" width="0.1524" layer="91"/>
 <wire x1="81.28" y1="33.02" x2="78.74" y2="33.02" width="0.1524" layer="91"/>
-<pinref part="D1" gate="G$1" pin="A"/>
+<pinref part="D2" gate="G$1" pin="A"/>
 <wire x1="78.74" y1="43.18" x2="81.28" y2="43.18" width="0.1524" layer="91"/>
 <junction x="81.28" y="43.18"/>
@@
 <pinref part="R5" gate="G$1" pin="2"/>
 <wire x1="88.9" y1="55.88" x2="88.9" y2="63.5" width="0.1524" layer="91"/>
-<pinref part="D3" gate="G$1" pin="A"/>
+<pinref part="D4" gate="G$1" pin="A"/>
 <wire x1="88.9" y1="63.5" x2="88.9" y2="68.58" width="0.1524" layer="91"/>
 <wire x1="99.06" y1="63.5" x2="88.9" y2="63.5" width="0.1524" layer="91"/>
@@
 <net name="N$5" class="0">
 <segment>
-<pinref part="D4" gate="G$1" pin="C"/>
+<pinref part="D3" gate="G$1" pin="C"/>
 <pinref part="R5" gate="G$1" pin="1"/>
 <wire x1="99.06" y1="68.58" x2="99.06" y2="73.66" width="0.1524" layer="91"/>
@@
 <net name="N$7" class="0">
 <segment>
-<pinref part="D4" gate="G$1" pin="A"/>
-<pinref part="D3" gate="G$1" pin="C"/>
+<pinref part="D3" gate="G$1" pin="A"/>
+<pinref part="D4" gate="G$1" pin="C"/>
 <wire x1="104.14" y1="68.58" x2="104.14" y2="63.5" width="0.1524" layer="91"/>
 <pinref part="IC1" gate="B" pin="OUT"/>
@@
 <wire x1="137.16" y1="55.88" x2="139.7" y2="55.88" width="0.1524" layer="91"/>
 <wire x1="137.16" y1="60.96" x2="121.92" y2="60.96" width="0.1524" layer="91"/>
-<pinref part="R7" gate="G$1" pin="1"/>
-<pinref part="R8" gate="G$1" pin="2"/>
-<wire x1="121.92" y1="60.96" x2="121.92" y2="50.8" width="0.1524" layer="91"/>
-<junction x="121.92" y="50.8"/>
 <junction x="137.16" y="60.96"/>
-<wire x1="121.92" y1="50.8" x2="129.54" y2="50.8" width="0.1524" layer="91"/>
-</segment>
-</net>
-<net name="N$10" class="0">
-<segment>
-<pinref part="IC2" gate="G$1" pin="REFADJ"/>
 <pinref part="R7" gate="G$1" pin="2"/>
 </segment>
@@
 </segment>
 </net>
+<net name="N$21" class="0">
+<segment>
+<pinref part="R7" gate="G$1" pin="1"/>
+<pinref part="R8" gate="G$1" pin="2"/>
+<pinref part="IC2" gate="G$1" pin="REFADJ"/>
+<wire x1="121.92" y1="50.8" x2="139.7" y2="50.8" width="0.1524" layer="91"/>
+<junction x="121.92" y="50.8"/>
+</segment>
+</net>
