File: ETI vocoder/output amp.brd (EAGLE design)
At the start: 82.9 x 32.7 mm, 18 parts, among them IC1 LM1458N, IC2 LM741P, J1 22-23-2031, X2 22-23-2051, X3 22-23-2021

Commit message: All ETI boards checked for caps and pots
Connections:
- net RETURN renamed FX_RETURN
Routing:
- net SPEECH: track 37.3 -> 41.1 mm
- net MIX: track 21.7 -> 18.2 mm
- net +12V: track 41.0 -> 43.5 mm
- net EXT_EXCIT: track 45.4 -> 47.5 mm
- net -12V: vias 0 -> 1
Other:
- board text added: "+12V"
- board text added: "-12V"
- board text added: "Ch1"
- board text added: "Ch3"
- board text added: "ETI Vocoder"
- board text added: "Ext exc bp"
- board text added: "Fx ret"
- board text added: "Out"
- board text added: "Output v1.0"
- board text added: "Speech bp"
- board text added: "To fx"
- board text removed: "ETI vocoder"
- board text removed: "Output board"
- board text removed: "Rev 1.0"
- board text removed: "Xonik Devices"
Changed lines of the file:
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@@
 <?xml version="1.0" encoding="utf-8"?>
 <!DOCTYPE eagle SYSTEM "eagle.dtd">
-<eagle version="7.2.0">
+<eagle version="6.2">
 <drawing>
 <settings>
@@
 <setting verticaltext="up"/>
 </settings>
-<grid distance="0.0125" unitdist="inch" unit="mm" style="dots" multiple="1" display="yes" altdistance="0.025" altunitdist="inch" altunit="inch"/>
+<grid distance="0.0125" unitdist="inch" unit="inch" style="dots" multiple="1" display="yes" altdistance="0.025" altunitdist="inch" altunit="inch"/>
 <layers>
 <layer number="1" name="Top" color="4" fill="1" visible="yes" active="yes"/>
@@
 <layer number="25" name="tNames" color="7" fill="1" visible="yes" active="yes"/>
 <layer number="26" name="bNames" color="7" fill="1" visible="yes" active="yes"/>
-<layer number="27" name="tValues" color="7" fill="1" visible="yes" active="yes"/>
-<layer number="28" name="bValues" color="7" fill="1" visible="yes" active="yes"/>
+<layer number="27" name="tValues" color="7" fill="1" visible="no" active="yes"/>
+<layer number="28" name="bValues" color="7" fill="1" visible="no" active="yes"/>
 <layer number="29" name="tStop" color="7" fill="3" visible="no" active="yes"/>
 <layer number="30" name="bStop" color="7" fill="6" visible="no" active="yes"/>
@@
 <wire x1="6.0325" y1="24.765" x2="4.7625" y2="24.765" width="0.254" layer="25"/>
 <text x="43.4975" y="24.4475" size="1.27" layer="25" font="vector">GND</text>
-<text x="53.975" y="0.9525" size="1.27" layer="25" font="vector" rot="R90">ETI vocoder</text>
-<text x="56.1975" y="0.9525" size="1.27" layer="25" font="vector" rot="R90">Output board</text>
-<text x="58.42" y="0.9525" size="1.27" layer="25" font="vector" rot="R90">Rev 1.0</text>
-<text x="60.6425" y="0.9525" size="1.27" layer="25" font="vector" rot="R90">Xonik Devices</text>
+<text x="3.81" y="27.305" size="1.016" layer="26" font="vector" rot="MR270">GND</text>
+<text x="6.35" y="27.305" size="1.016" layer="26" font="vector" rot="MR270">Out</text>
+<text x="11.43" y="27.305" size="1.016" layer="26" font="vector" rot="MR270">To fx</text>
+<text x="8.89" y="27.305" size="1.016" layer="26" font="vector" rot="MR270">Fx ret</text>
+<text x="27.6225" y="24.4475" size="1.016" layer="26" font="vector" rot="MR270">-12V</text>
+<text x="22.86" y="24.4475" size="1.016" layer="26" font="vector" rot="MR270">GND</text>
+<text x="17.78" y="24.4475" size="1.016" layer="26" font="vector" rot="MR270">+12V</text>
+<text x="45.085" y="27.305" size="1.016" layer="26" font="vector" rot="MR270">GND</text>
+<text x="42.545" y="27.6225" size="1.016" layer="26" font="vector" rot="MR270">Ch1</text>
+<text x="40.005" y="27.6225" size="1.016" layer="26" font="vector" rot="MR270">Ch3</text>
+<text x="30.7975" y="29.21" size="1.016" layer="26" font="vector" rot="MR270">Speech bp</text>
+<text x="32.7025" y="27.6225" size="1.016" layer="26" font="vector" rot="MR270">Ext exc bp</text>
+<wire x1="33.3375" y1="25.7175" x2="36.195" y2="25.7175" width="0.254" layer="26"/>
+<wire x1="36.195" y1="25.7175" x2="36.83" y2="26.3525" width="0.254" layer="26"/>
+<wire x1="36.83" y1="26.3525" x2="36.83" y2="26.9875" width="0.254" layer="26"/>
+<wire x1="36.83" y1="26.9875" x2="36.5125" y2="26.9875" width="0.254" layer="26"/>
+<wire x1="36.5125" y1="26.9875" x2="36.83" y2="27.305" width="0.254" layer="26"/>
+<wire x1="36.83" y1="27.305" x2="37.1475" y2="26.9875" width="0.254" layer="26"/>
+<wire x1="37.1475" y1="26.9875" x2="36.83" y2="26.9875" width="0.254" layer="26"/>
+<wire x1="30.7975" y1="29.21" x2="32.7025" y2="29.21" width="0.254" layer="26"/>
+<wire x1="32.7025" y1="29.21" x2="32.7025" y2="29.5275" width="0.254" layer="26"/>
+<wire x1="32.7025" y1="29.5275" x2="33.02" y2="29.21" width="0.254" layer="26"/>
+<wire x1="33.02" y1="29.21" x2="32.7025" y2="28.8925" width="0.254" layer="26"/>
+<wire x1="32.7025" y1="28.8925" x2="32.7025" y2="29.21" width="0.254" layer="26"/>
+<text x="21.59" y="7.62" size="1.016" layer="25" font="vector">ETI Vocoder</text>
+<text x="21.59" y="5.715" size="1.016" layer="25" font="vector">Output v1.0</text>
 </plain>
 <attributes>
@@
 </class>
 </classes>
-<designrules name="default">
+<designrules>
 <description language="de">&lt;b&gt;EAGLE Design Rules&lt;/b&gt;
 &lt;p&gt;
@@
 <pass name="Default">
 <param name="RoutingGrid" value="50mil"/>
-<param name="AutoGrid" value="1"/>
-<param name="Efforts" value="0"/>
-<param name="TopRouterVariant" value="1"/>
 <param name="tpViaShape" value="round"/>
-<param name="PrefDir.1" value="a"/>
+<param name="PrefDir.1" value="|"/>
 <param name="PrefDir.2" value="0"/>
 <param name="PrefDir.3" value="0"/>
@@
 <param name="PrefDir.14" value="0"/>
 <param name="PrefDir.15" value="0"/>
-<param name="PrefDir.16" value="a"/>
+<param name="PrefDir.16" value="-"/>
 <param name="cfVia" value="8"/>
 <param name="cfNonPref" value="5"/>
@@
 <contactref element="IC2" pad="6"/>
 <contactref element="R6" pad="2"/>
-<wire x1="14.605" y1="13.6525" x2="14.605" y2="24.765" width="0.6096" layer="1"/>
-<wire x1="14.605" y1="24.765" x2="13.335" y2="26.035" width="0.6096" layer="1"/>
+<wire x1="14.605" y1="13.6525" x2="14.605" y2="16.8275" width="0.6096" layer="1"/>
 <wire x1="9.525" y1="23.495" x2="9.525" y2="24.765" width="0.6096" layer="1"/>
 <wire x1="9.525" y1="24.765" x2="10.795" y2="26.035" width="0.6096" layer="1"/>
-<wire x1="10.795" y1="26.035" x2="13.335" y2="26.035" width="0.6096" layer="1"/>
 <contactref element="J1" pad="2"/>
 <wire x1="10.795" y1="26.035" x2="10.795" y2="29.21" width="0.6096" layer="1"/>
+<wire x1="14.605" y1="16.8275" x2="9.525" y2="21.9075" width="0.6096" layer="1"/>
+<wire x1="9.525" y1="21.9075" x2="9.525" y2="23.495" width="0.6096" layer="1"/>
 </signal>
 <signal name="N$10">
@@
 <wire x1="34.29" y1="23.495" x2="34.29" y2="21.59" width="0.6096" layer="16"/>
 <wire x1="34.29" y1="21.59" x2="17.78" y2="21.59" width="0.6096" layer="16"/>
-<wire x1="17.4625" y1="19.685" x2="17.4625" y2="26.5025" width="0.6096" layer="1"/>
 <wire x1="17.4625" y1="26.5025" x2="18.265" y2="27.305" width="0.6096" layer="1"/>
 <wire x1="6.985" y1="23.495" x2="6.985" y2="21.59" width="0.6096" layer="16"/>
 <wire x1="6.985" y1="21.59" x2="17.78" y2="21.59" width="0.6096" layer="16"/>
 <wire x1="17.78" y1="21.59" x2="17.4625" y2="19.685" width="0.6096" layer="16"/>
+<wire x1="17.4625" y1="26.5025" x2="17.4625" y2="19.685" width="0.6096" layer="1"/>
+<wire x1="17.4625" y1="19.685" x2="14.9225" y2="19.685" width="0.6096" layer="1"/>
 </signal>
 <signal name="-12V">
@@
 <wire x1="26.9875" y1="26.52" x2="26.185" y2="27.305" width="0.6096" layer="1"/>
 <wire x1="23.1775" y1="15.875" x2="26.9875" y2="19.685" width="0.6096" layer="16"/>
-<wire x1="26.9875" y1="19.685" x2="41.91" y2="19.685" width="0.6096" layer="16"/>
+<wire x1="26.9875" y1="19.685" x2="29.5275" y2="19.685" width="0.6096" layer="16"/>
+<wire x1="29.5275" y1="19.685" x2="41.91" y2="19.685" width="0.6096" layer="16"/>
+<via x="29.5275" y="19.685" extent="1-16" drill="0.8" diameter="1.6764"/>
 </signal>
 <signal name="SPEECH">
@@
 <wire x1="18.0975" y1="14.2875" x2="24.4475" y2="14.2875" width="0.6096" layer="16"/>
 <via x="24.4475" y="14.2875" extent="1-16" drill="0.8"/>
-<wire x1="24.4475" y1="14.2875" x2="29.21" y2="19.05" width="0.6096" layer="1"/>
-<wire x1="29.21" y1="19.05" x2="29.21" y2="25.0825" width="0.6096" layer="1"/>
+<wire x1="24.4475" y1="14.2875" x2="27.305" y2="14.2875" width="0.6096" layer="1"/>
+<wire x1="27.305" y1="14.2875" x2="31.4325" y2="17.78" width="0.6096" layer="1"/>
+<wire x1="31.4325" y1="17.78" x2="31.4325" y2="20.6375" width="0.6096" layer="1"/>
+<wire x1="31.4325" y1="20.6375" x2="29.21" y2="22.86" width="0.6096" layer="1"/>
+<wire x1="29.21" y1="22.86" x2="29.21" y2="25.0825" width="0.6096" layer="1"/>
 <wire x1="29.21" y1="25.0825" x2="33.3375" y2="29.21" width="0.6096" layer="1"/>
 <wire x1="33.3375" y1="29.21" x2="34.29" y2="29.21" width="0.6096" layer="1"/>
@@
 <wire x1="28.8925" y1="13.0175" x2="31.75" y2="15.875" width="0.6096" layer="16"/>
 <via x="31.75" y="15.875" extent="1-16" drill="0.8"/>
-<wire x1="31.75" y1="15.875" x2="31.75" y2="24.13" width="0.6096" layer="1"/>
+<wire x1="31.75" y1="15.875" x2="34.29" y2="18.415" width="0.6096" layer="1"/>
+<wire x1="34.29" y1="18.415" x2="34.29" y2="20.0025" width="0.6096" layer="1"/>
+<wire x1="34.29" y1="20.0025" x2="31.75" y2="22.5425" width="0.6096" layer="1"/>
+<wire x1="31.75" y1="22.5425" x2="31.75" y2="24.13" width="0.6096" layer="1"/>
 <wire x1="31.75" y1="24.13" x2="33.02" y2="25.4" width="0.6096" layer="1"/>
 <wire x1="33.02" y1="25.4" x2="35.56" y2="25.4" width="0.6096" layer="1"/>
@@
 <wire x1="46.99" y1="13.97" x2="45.085" y2="15.875" width="0.6096" layer="1"/>
 </signal>
-<signal name="RETURN">
+<signal name="FX_RETURN">
 <contactref element="J1" pad="1"/>
 <contactref element="X3" pad="2"/>
 <wire x1="5.715" y1="29.21" x2="8.255" y2="29.21" width="0.6096" layer="16"/>
 </signal>
+<signal name="N$2">
+<via x="14.9225" y="19.685" extent="1-16" drill="0.8" diameter="1.6764"/>
+</signal>
 </signals>
