File: ETI vocoder/slew rate control.sch (EAGLE design)
At the start: 28 parts, among them CN1 NMJ6HCD2, IC1 LM556N, Q1 2N3904, Q2 2N3906, X1 22-23-2031

Commit message: Fixed input boards in regards to article and added spacer holes
Parts:
- C2: device resistor:C-EU050-025X075 -> resistor:C-EU075-032X103
- C4: device resistor:C-EU025-025X050 -> resistor:C-EU025_050-025X075
Connections:
- net FROM_V/UV_SWITCH: now also CN1.TIP; no longer CN1.SLEEVE
- net N$13: now also CN1.SLEEVE; no longer CN1.TIP
Other:
- note added: "Sjekket bein på jack"
- note added: "Sjekket footprint på caps"
- note added: "Sjekket retning på pot"
- note removed: "Sjekk bein på jack - denne er ring make, altså at ring lukkes, ikke åpnes, når jack settes inn."
- note removed: "Sjekk retning på pot"
Changed lines of the file:
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@@
 <?xml version="1.0" encoding="utf-8"?>
 <!DOCTYPE eagle SYSTEM "eagle.dtd">
-<eagle version="7.2.0">
+<eagle version="6.2">
 <drawing>
 <settings>
@@
 <layers>
 <layer number="1" name="Top" color="4" fill="1" visible="no" active="no"/>
+<layer number="2" name="Route2" color="1" fill="3" visible="no" active="no"/>
+<layer number="3" name="Route3" color="4" fill="3" visible="no" active="no"/>
+<layer number="14" name="Route14" color="1" fill="6" visible="no" active="no"/>
+<layer number="15" name="Route15" color="4" fill="6" visible="no" active="no"/>
 <layer number="16" name="Bottom" color="1" fill="1" visible="no" active="no"/>
 <layer number="17" name="Pads" color="2" fill="1" visible="no" active="no"/>
@@
 <part name="R13" library="resistor" deviceset="R-EU_" device="0207/7" value="1k"/>
 <part name="C1" library="resistor" deviceset="C-EU" device="025-025X050" value="10n"/>
-<part name="C2" library="resistor" deviceset="C-EU" device="050-025X075" value="33n"/>
+<part name="C2" library="resistor" deviceset="C-EU" device="075-032X103" value="33n"/>
 <part name="C3" library="resistor" deviceset="C-EU" device="025-025X050" value="100p"/>
-<part name="C4" library="resistor" deviceset="C-EU" device="025-025X050" value="560p"/>
+<part name="C4" library="resistor" deviceset="C-EU" device="025_050-025X075" value="560p"/>
 <part name="C5" library="resistor" deviceset="C-EU" device="025-025X050" value="10n"/>
 <part name="C6" library="resistor" deviceset="CPOL-EU" device="E2.5-5" value="22u"/>
@@
 <sheet>
 <plain>
-<text x="58.42" y="66.04" size="1.778" layer="91">Sjekk retning på pot</text>
-<text x="83.82" y="-33.02" size="1.778" layer="91">Sjekk bein på jack - denne er ring make, altså at ring lukkes, ikke åpnes, når jack settes inn.</text>
+<text x="83.82" y="-38.1" size="1.778" layer="91">Sjekket retning på pot</text>
+<text x="83.82" y="-33.02" size="1.778" layer="91">Sjekket bein på jack</text>
+<text x="83.82" y="-43.18" size="1.778" layer="91">Sjekket footprint på caps</text>
 </plain>
 <instances>
@@
 <net name="FROM_V/UV_SWITCH" class="0">
 <segment>
-<pinref part="CN1" gate="G$1" pin="SLEEVE"/>
-<wire x1="101.6" y1="-5.08" x2="116.84" y2="-5.08" width="0.1524" layer="91"/>
-<label x="101.6" y="-5.08" size="1.778" layer="95"/>
+<wire x1="101.6" y1="-17.78" x2="127" y2="-17.78" width="0.1524" layer="91"/>
+<label x="104.14" y="-17.78" size="1.778" layer="95"/>
+<pinref part="CN1" gate="G$1" pin="TIP"/>
+<junction x="101.6" y="-17.78"/>
 </segment>
 <segment>
@@
 <net name="N$13" class="0">
 <segment>
-<pinref part="CN1" gate="G$1" pin="TIP"/>
-<wire x1="101.6" y1="-17.78" x2="132.08" y2="-17.78" width="0.1524" layer="91"/>
 <pinref part="R12" gate="G$1" pin="1"/>
-<wire x1="132.08" y1="5.08" x2="132.08" y2="-17.78" width="0.1524" layer="91"/>
-</segment>
-</net>
+<pinref part="CN1" gate="G$1" pin="SLEEVE"/>
+<wire x1="132.08" y1="5.08" x2="132.08" y2="-5.08" width="0.1524" layer="91"/>
+<wire x1="132.08" y1="-5.08" x2="101.6" y2="-5.08" width="0.1524" layer="91"/>
+</segment>
+</net>

Commit message: Finished first of two halves of the universal voice board
Changed lines of the file:
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@@
 <wire x1="119.38" y1="48.26" x2="124.46" y2="48.26" width="0.1524" layer="91"/>
 <pinref part="RV1" gate="G$1" pin="1S"/>
+<wire x1="124.46" y1="53.34" x2="124.46" y2="48.26" width="0.1524" layer="91"/>
 <wire x1="124.46" y1="48.26" x2="129.54" y2="48.26" width="0.1524" layer="91"/>
 <junction x="119.38" y="48.26"/>
-<junction x="124.46" y="48.26"/>
+<junction x="124.46" y="53.34"/>
 <junction x="129.54" y="48.26"/>
 </segment>
@@
 <wire x1="124.46" y1="27.94" x2="134.62" y2="27.94" width="0.1524" layer="91"/>
 <pinref part="RV1" gate="G$1" pin="1A"/>
-<wire x1="134.62" y1="27.94" x2="134.62" y2="48.26" width="0.1524" layer="91"/>
+<wire x1="134.62" y1="27.94" x2="134.62" y2="53.34" width="0.1524" layer="91"/>
 </segment>
 </net>
