File: ETI vocoder/internal excitation 2 w gp.brd (EAGLE design)
At the start: 94 x 53.6 mm, 56 parts, among them IC10 LM1458N, IC11 LM1458N, IC12 4016N, IC2 LM1458N, IC3 TL081P, IC8 TL082P, IC9 CA3080E, Q2 BC212L, Q3 BC182L, Q4 BC212L

Commit message: Finished second combined board, only missing break-aparts
Routing:
- net +12V: track 149.9 -> 134.1 mm
- net N$13: track 27.3 -> 33.0 mm
- net N$25: track 20.8 -> 21.5 mm
Other:
- outline, holes or cut-outs redrawn
Changed lines of the file:
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@@
 <setting verticaltext="up"/>
 </settings>
-<grid distance="0.005" unitdist="inch" unit="inch" style="dots" multiple="1" display="yes" altdistance="0.025" altunitdist="inch" altunit="inch"/>
+<grid distance="0.0125" unitdist="inch" unit="inch" style="dots" multiple="1" display="yes" altdistance="0.025" altunitdist="inch" altunit="inch"/>
 <layers>
 <layer number="1" name="Top" color="4" fill="1" visible="yes" active="yes"/>
@@
 <wire x1="31.115" y1="12.065" x2="31.115" y2="0" width="0" layer="20"/>
 <wire x1="31.115" y1="0" x2="85.725" y2="0" width="0" layer="20"/>
-<wire x1="85.725" y1="0" x2="85.725" y2="10.795" width="0" layer="20"/>
-<wire x1="85.725" y1="10.795" x2="86.995" y2="12.065" width="0" layer="20" curve="-90"/>
-<wire x1="86.995" y1="12.065" x2="93.96" y2="12.065" width="0" layer="20"/>
-<wire x1="93.96" y1="12.065" x2="93.96" y2="53.645" width="0" layer="20"/>
+<wire x1="85.725" y1="0" x2="85.725" y2="13.6525" width="0" layer="20"/>
+<wire x1="85.725" y1="13.6525" x2="86.995" y2="14.9225" width="0" layer="20" curve="-90"/>
+<wire x1="86.995" y1="14.9225" x2="93.96" y2="14.9225" width="0" layer="20"/>
+<wire x1="93.96" y1="14.9225" x2="93.96" y2="53.645" width="0" layer="20"/>
 <wire x1="93.96" y1="53.645" x2="0" y2="53.645" width="0" layer="20"/>
 <wire x1="0" y1="53.645" x2="0" y2="0" width="0" layer="20"/>
@@
 <wire x1="2.54" y1="41.91" x2="2.54" y2="49.38" width="0.6096" layer="1"/>
 <wire x1="2.54" y1="49.38" x2="2.39" y2="48.26" width="0.6096" layer="1"/>
-<wire x1="19.05" y1="41.91" x2="19.05" y2="43.18" width="0.6096" layer="16"/>
-<wire x1="19.05" y1="43.18" x2="22.225" y2="46.355" width="0.6096" layer="16"/>
-<wire x1="22.225" y1="46.355" x2="30.48" y2="46.355" width="0.6096" layer="16"/>
-<wire x1="30.48" y1="46.355" x2="31.75" y2="47.625" width="0.6096" layer="16"/>
 <contactref element="IC9" pad="7"/>
 <wire x1="80.01" y1="25.4" x2="80.01" y2="22.86" width="0.6096" layer="16"/>
@@
 <wire x1="72.39" y1="4.445" x2="74.295" y2="6.35" width="0.6096" layer="16"/>
 <wire x1="74.295" y1="6.35" x2="76.835" y2="6.35" width="0.6096" layer="16"/>
-<wire x1="76.835" y1="6.35" x2="78.105" y2="7.62" width="0.6096" layer="16"/>
-<wire x1="78.105" y1="7.62" x2="81.28" y2="7.62" width="0.6096" layer="16"/>
-<wire x1="81.28" y1="7.62" x2="83.82" y2="10.16" width="0.6096" layer="16"/>
-<wire x1="83.82" y1="10.16" x2="83.82" y2="13.335" width="0.6096" layer="16"/>
-<wire x1="83.82" y1="13.335" x2="84.455" y2="13.97" width="0.6096" layer="16"/>
-<wire x1="84.455" y1="13.97" x2="88.265" y2="13.97" width="0.6096" layer="16"/>
-<wire x1="88.265" y1="13.97" x2="91.44" y2="17.78" width="0.6096" layer="16"/>
+<wire x1="76.835" y1="6.35" x2="78.74" y2="8.255" width="0.6096" layer="16"/>
+<wire x1="78.74" y1="8.255" x2="78.74" y2="13.335" width="0.6096" layer="16"/>
+<wire x1="78.74" y1="13.335" x2="80.645" y2="15.24" width="0.6096" layer="16"/>
+<wire x1="80.645" y1="15.24" x2="85.4075" y2="15.24" width="0.6096" layer="16"/>
+<wire x1="85.4075" y1="15.24" x2="86.6775" y2="16.51" width="0.6096" layer="16"/>
+<wire x1="86.6775" y1="16.51" x2="86.6775" y2="19.05" width="0.6096" layer="16"/>
+<wire x1="86.6775" y1="19.05" x2="88.265" y2="20.6375" width="0.6096" layer="16"/>
+<wire x1="88.265" y1="20.6375" x2="90.17" y2="20.6375" width="0.6096" layer="16"/>
+<wire x1="90.17" y1="20.6375" x2="91.44" y2="19.3675" width="0.6096" layer="16"/>
+<wire x1="91.44" y1="19.3675" x2="91.44" y2="17.78" width="0.6096" layer="16"/>
 </signal>
 <signal name="BOARD2_MIX">
@@
 <contactref element="R36" pad="1"/>
 <contactref element="IC9" pad="3"/>
-<wire x1="76.2" y1="8.255" x2="78.74" y2="10.795" width="0.6096" layer="16"/>
-<wire x1="78.74" y1="10.795" x2="78.74" y2="13.335" width="0.6096" layer="16"/>
-<wire x1="78.74" y1="13.335" x2="80.645" y2="15.24" width="0.6096" layer="16"/>
-<wire x1="80.645" y1="15.24" x2="82.55" y2="15.24" width="0.6096" layer="16"/>
-<wire x1="82.55" y1="15.24" x2="82.55" y2="17.78" width="0.6096" layer="16"/>
-<wire x1="88.265" y1="17.78" x2="88.265" y2="16.51" width="0.6096" layer="16"/>
-<wire x1="88.265" y1="16.51" x2="86.995" y2="15.24" width="0.6096" layer="16"/>
-<wire x1="86.995" y1="15.24" x2="82.55" y2="15.24" width="0.6096" layer="16"/>
+<wire x1="76.2" y1="8.255" x2="78.74" y2="10.795" width="0.6096" layer="1"/>
+<wire x1="78.74" y1="10.795" x2="78.74" y2="13.335" width="0.6096" layer="1"/>
+<wire x1="78.74" y1="13.335" x2="82.55" y2="17.145" width="0.6096" layer="1"/>
+<wire x1="82.55" y1="17.78" x2="82.55" y2="20.32" width="0.6096" layer="1"/>
+<wire x1="82.55" y1="20.32" x2="85.725" y2="20.32" width="0.6096" layer="1"/>
+<wire x1="85.725" y1="20.32" x2="88.265" y2="17.78" width="0.6096" layer="1"/>
+<wire x1="82.55" y1="17.78" x2="82.55" y2="17.145" width="0.6096" layer="1"/>
 </signal>
 <signal name="N$26">
