File: ETI vocoder/internal excitation 2 w gp.brd (EAGLE design)
At the start: 94 x 53.6 mm, 56 parts, among them IC10 LM1458N, IC11 LM1458N, IC12 4016N, IC2 LM1458N, IC3 TL081P, IC8 TL082P, IC9 CA3080E, Q2 BC212L, Q3 BC182L, Q4 BC212L

Commit message: Fixed wrong value for C11/C15 on internal excitation board (should be 220uF, not 22uF)
Parts:
- C11: value 22n -> 220n
Changed lines of the file:
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@@
 <attribute name="VALUE" x="64.8462" y="40.386" size="1.27" layer="27" ratio="10" rot="R270"/>
 </element>
-<element name="C11" library="resistor" package="C050-025X075" value="22n" x="6.35" y="29.21" smashed="yes">
+<element name="C11" library="resistor" package="C050-025X075" value="220n" x="6.35" y="29.21" smashed="yes">
 <attribute name="NAME" x="9.906" y="32.131" size="1.27" layer="25" ratio="10" rot="R180"/>
 <attribute name="VALUE" x="4.064" y="26.416" size="1.27" layer="27" ratio="10"/>
