File: ETI vocoder/internal excitation w gp.sch (EAGLE design)
At the start: 51 parts, among them IC1 LM1458N, IC3 TL081P, IC4 UA741P, IC5 4006N, IC6 4030N, IC7 LM1458N, Q1 BC182L

Commit message: Updated trimpot names and positions
Parts:
- C1, C6, C8: device resistor:C-EU075-032X103 -> resistor:C-EU050-030X075
Changed lines of the file:
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@@
 <part name="GND2" library="supply1" deviceset="GND" device=""/>
 <part name="GND3" library="supply1" deviceset="GND" device=""/>
-<part name="C1" library="resistor" deviceset="C-EU" device="075-032X103" value="100n"/>
+<part name="C1" library="resistor" deviceset="C-EU" device="050-030X075" value="100n"/>
 <part name="RV5" library="joakim" deviceset="POT16_W_BRACKET" device="&quot;&quot;" value="10k"/>
 <part name="PR4" library="pot" deviceset="TRIM_EU-" device="CA9V" value="2k2"/>
@@
 <part name="R23" library="resistor" deviceset="R-EU_" device="0207/7" value="27k"/>
 <part name="R22" library="resistor" deviceset="R-EU_" device="0207/7" value="330k"/>
-<part name="C8" library="resistor" deviceset="C-EU" device="075-032X103" value="10n"/>
-<part name="C6" library="resistor" deviceset="C-EU" device="075-032X103" value="33n"/>
+<part name="C8" library="resistor" deviceset="C-EU" device="050-030X075" value="10n"/>
+<part name="C6" library="resistor" deviceset="C-EU" device="050-030X075" value="33n"/>
 <part name="C5" library="resistor" deviceset="C-EU" device="025-025X050" value="220p"/>
 <part name="C7" library="resistor" deviceset="C-EU" device="025-025X050" value="100p"/>
