File: ETI vocoder/internal excitation 2.sch (EAGLE design)
At the start: 55 parts, among them IC1 CA3080E, IC10 LM1458N, IC11 LM1458N, IC12 4016N, IC2 LM1458N, IC3 TL081P, IC4 TL082P, Q2 BC212L, Q3 BC182L, Q4 BC212L

Commit message: Fixed input boards in regards to article and added spacer holes
Parts:
- removed CARD1: (no value), con-molex:22-23-2061
- removed IC1: CA3080E, synthdiy:CA3080E
- added BOARD2: 22-23-2041, con-molex:22-23-2041
- added BOARD2-PWR: 22-23-2021, con-molex:22-23-2021
- added IC9: CA3080E, joakim:CA3080E
- C10: device resistor:C-EU025-025X050 -> resistor:C-EU075-032X103
- C11, C12: device resistor:C-EU025-025X050 -> resistor:C-EU050-025X075
- C3: device resistor:C-EU050-025X075 -> resistor:C-EU075-032X103
- C4: value 100n -> 10n
- R6: device resistor:R-EU_0207/7 -> resistor:R-EU_0207/10
- renumbered IC4 to IC8
Connections:
- removed net N$29: Q2.E, R34.1
- removed net N$33: IC1.OUT, PR3.E
- removed net OUTPUT: IC12A.B, IC12C.B
- new net N$22: IC9G$1.OUT, PR3.A
- new net N$24: Q2.C, R34.1
- net +12V: now also IC9G$2.V+, PR2.A; no longer IO-1.S, PR2.E
- net -12V: now also IC9G$2.V-, IO-5.S, PR2.E; no longer PR2.A
- net 2KHZ: now also IO-1.S; no longer IO-8.S
- net 4KHZ: now also IO-2.S; no longer IO-7.S
- net BOARD2_MIX: now also BOARD2-4.S; no longer CARD1-4.S
- net EXT_EXCIT: now also IO-8.S; no longer IO-4.S
- net GND: now also PR3.E, RV6G$1.1E; no longer PR3.A, RV6G$1.1A
- net N$25: now also IC9G$1.+IN; no longer IC1.+IN
- net N$26: now also IC9G$1.-IN; no longer IC1.-IN
- net N$28: now also IC9G$1.IABC; no longer IC1.IABC
- net N$30: now also Q2.E; no longer Q2.C
- net N$9: now also RV6G$1.1A; no longer RV6G$1.1E
- net OUT: now also IC12A.B, IC12C.B, IO-7.S; no longer IO-5.S
- net VCA_CTRL: now also BOARD2-2.S; no longer CARD1-2.S
- net VCA_SIGNAL: now also BOARD2-3.S; no longer CARD1-1.S
- net VDD: now also BOARD2-PWR-2.S; no longer CARD1-5.S
- net VSS: now also BOARD2-PWR-1.S; no longer CARD1-6.S
- net V_UV_ON_OFF: now also IO-4.S; no longer IO-2.S
- net X: now also BOARD2-1.S; no longer CARD1-3.S
Other:
- note added: "Kondensatorer sjekket"
- note added: "Pots er sjekket"
- note added: "Sjekket mot artikkeø"
- note removed: "Sjekk retning på pots!"
- note removed: "Vurdere å flytte switch output til foran på board"
- moved on the sheet: IO-1, IO-2, IO-3, IO-4, IO-5, IO-6, IO-7, IO-8, PR2, PR3, Q2, RV6

Commit message: Various updates while working on the real vocoder
Other:
- note added: "Error: c11 is 22n in schematics and 220n in parts list"
Changed lines of the file:
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@@
 <?xml version="1.0" encoding="utf-8"?>
 <!DOCTYPE eagle SYSTEM "eagle.dtd">
-<eagle version="6.2">
+<eagle version="6.5.0">
 <drawing>
 <settings>
@@
 <text x="-17.78" y="180.34" size="5.08" layer="91">Kondensatorer sjekket</text>
 <text x="-17.78" y="198.12" size="1.778" layer="91">Sjekket mot artikkeø</text>
+<text x="-33.02" y="142.24" size="1.778" layer="97">Error: c11 is 22n in schematics and 220n in parts list</text>
 </plain>
 <instances>
