File: ETI vocoder/led ppm display w gp.sch (EAGLE design)
At the start: 29 parts, among them IC1 TL082P, IC2 LM3915N

Commit message: Various updates while working on the real vocoder
Other:
- note added: "The shown combination of R7 and R8 will give an approximate led current of 18.3mA (using the formulas in the LM3915 datasheet."
Changed lines of the file:
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@@
 <text x="187.96" y="50.8" size="1.778" layer="97" rot="R90">Green</text>
 <text x="106.68" y="81.28" size="1.778" layer="97">R7 is misplaced in the schematics in the original article</text>
+<text x="129.54" y="2.54" size="1.778" layer="97">The shown combination of R7 and R8
+will give an approximate led current
+of 18.3mA (using the formulas in
+the LM3915 datasheet.</text>
 </plain>
 <instances>
