File: ETI vocoder/Combined-4-ordered-080117.brd (EAGLE design)
At the start: 92.9 x 100 mm, 117 parts, among them IC1 TL082P, IC10 LM1458N, IC11 LM1458N, IC12 4016N, IC2 LM3915N, IC3 LM4558N, IC4 LM1458N, IC5 LM1458N, IC6 TL081P, IC8 TL082P, IC9 CA3080E, Q2 BC212L, Q3 BC182L, Q4 BC212L

Commit message: Fixed wrong value for C11/C15 on internal excitation board (should be 220uF, not 22uF)
Parts:
- C15: value 22n -> 220n
Changed lines of the file:
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@@
 <attribute name="VALUE" x="79.611" y="34.9963" size="1.27" layer="27" ratio="10" rot="R180"/>
 </element>
-<element name="C15" library="resistor" package="C050-025X075" value="22n" x="68.435" y="93.4925" smashed="yes" rot="R270">
+<element name="C15" library="resistor" package="C050-025X075" value="220n" x="68.435" y="93.4925" smashed="yes" rot="R270">
 <attribute name="NAME" x="71.356" y="89.9365" size="1.27" layer="25" ratio="10" rot="R90"/>
 <attribute name="VALUE" x="65.641" y="95.7785" size="1.27" layer="27" ratio="10" rot="R270"/>
