File: DCO/DCO.brd (EAGLE design)
At the start: 71.7 x 19.7 mm, 23 parts, among them IC1 PIC16F18325SL, IC2 MAX5216, IC3 TL082D, Q1 MMBT3906

Commit message: Cleanup
Parts:
- moved SV3 25.7 mm to (42.5, 11.4)
- moved R3 2.01 mm to (21.0, 16.8), turned to 90 degrees
- moved R2 1.62 mm to (23.2, 16.8), turned to 90 degrees
- moved C1 0.90 mm to (18.7, 16.8)
- moved C6 0.64 mm to (3.17, 16.8)
- moved C7 0.64 mm to (16.5, 16.8)
- moved Q1 0.63 mm to (27.0, 17.8)
Routing:
- net AGND: track 37.8 -> 33.2 mm
- net N$2: track 3.06 -> 5.67 mm
- net OSC1: track 9.66 -> 8.58 mm
- net N$3: track 3.02 -> 4.02 mm
- net DAC_REF: track 11.9 -> 12.9 mm
- net N$4: track 4.91 -> 5.86 mm
- net CAP1: track 23.8 -> 22.9 mm
- net TIMER_OUT: track 18.4 -> 17.8 mm
- net OSC2: track 12.7 -> 12.1 mm
Other:
- board size 71.7 x 19.7 mm -> 45.7 x 19.7 mm

Commit message: Cleanup
Parts:
- moved R4 2.01 mm to (28.9, 16.8), turned to 90 degrees
- moved Q1 1.35 mm to (26.0, 16.8), turned to 0 degrees
Routing:
- net N$2: track 5.67 -> 2.32 mm
- net CAP2: track 20.7 -> 23.5 mm
- net CAP1: track 22.9 -> 21.4 mm
Changed lines of the file:
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@@
 <attribute name="MF" value="MICROCHIP" x="-9.2075" y="14.605" size="1.778" layer="27" rot="R180" display="off"/>
 <attribute name="OC_FARNELL" value="9760520" x="-9.2075" y="14.605" size="1.778" layer="27" rot="R180" display="off"/>
-<attribute name="NAME" x="5.715" y="8.0645" size="1.27" layer="25"/>
+<attribute name="NAME" x="6.0325" y="8.0645" size="1.27" layer="25"/>
 <attribute name="VALUE" x="4.0005" y="11.43" size="1.27" layer="27" rot="R270"/>
 </element>
@@
 <attribute name="VALUE" x="15.8265" y="11.811" size="1.27" layer="27" rot="R270"/>
 </element>
-<element name="Q1" library="transistor-pnp" package="SOT23-BEC" value="MMBT3906" x="26.9875" y="17.78" smashed="yes" rot="R270">
-<attribute name="NAME" x="28.8925" y="19.3675" size="1.27" layer="25" rot="R270"/>
-<attribute name="VALUE" x="23.8125" y="19.685" size="1.27" layer="27" rot="R270"/>
+<element name="Q1" library="transistor-pnp" package="SOT23-BEC" value="MMBT3906" x="26.035" y="16.8275" smashed="yes">
+<attribute name="NAME" x="27.94" y="14.9225" size="1.27" layer="25" rot="R180"/>
+<attribute name="VALUE" x="24.13" y="13.6525" size="1.27" layer="27"/>
 </element>
 <element name="IC3" library="linear" package="SO08" value="TL082D" x="25.4" y="9.525" smashed="yes" rot="R180">
@@
 <attribute name="VALUE" x="23.241" y="16.0655" size="1.27" layer="27" rot="R90"/>
 </element>
-<element name="R4" library="resistor" package="R0805" value="2R2" x="28.2575" y="14.9225" smashed="yes">
-<attribute name="NAME" x="28.1305" y="12.446" size="1.27" layer="25"/>
-<attribute name="VALUE" x="27.4955" y="12.6365" size="1.27" layer="27"/>
+<element name="R4" library="resistor" package="R0805" value="2R2" x="28.8925" y="16.8275" smashed="yes" rot="R90">
+<attribute name="NAME" x="30.2895" y="13.9065" size="1.27" layer="25" rot="R180"/>
+<attribute name="VALUE" x="31.1785" y="16.0655" size="1.27" layer="27" rot="R90"/>
 </element>
 <element name="C1" library="resistor" package="C0805" value="270pF" x="18.7325" y="16.8275" smashed="yes" rot="R90">
@@
 </element>
 <element name="C2" library="resistor" package="C0805" value="100nF" x="29.5275" y="8.255" smashed="yes" rot="MR180">
-<attribute name="NAME" x="31.369" y="5.7785" size="1.27" layer="26" rot="MR0"/>
+<attribute name="NAME" x="31.0515" y="5.7785" size="1.27" layer="26" rot="MR0"/>
 <attribute name="VALUE" x="28.6385" y="10.541" size="1.27" layer="28" rot="MR180"/>
 </element>
 <element name="C3" library="resistor" package="C0805" value="100nF" x="29.5275" y="10.795" smashed="yes" rot="MR0">
-<attribute name="NAME" x="28.956" y="13.2715" size="1.27" layer="26" rot="MR180"/>
+<attribute name="NAME" x="31.0515" y="12.1285" size="1.27" layer="26" rot="MR0"/>
 <attribute name="VALUE" x="30.4165" y="8.509" size="1.27" layer="28" rot="MR0"/>
 </element>
@@
 </element>
 <element name="C6" library="resistor" package="C0805" value="" x="3.175" y="16.8275" smashed="yes" rot="R270">
-<attribute name="NAME" x="1.9685" y="13.3985" size="1.27" layer="25"/>
+<attribute name="NAME" x="3.7465" y="12.7635" size="1.27" layer="25" rot="R90"/>
 <attribute name="VALUE" x="0.889" y="17.7165" size="1.27" layer="27" rot="R270"/>
 </element>
@@
 <contactref element="Q1" pad="B"/>
 <contactref element="R2" pad="1"/>
-<wire x1="23.1775" y1="15.9775" x2="23.1775" y2="15.875" width="0.4064" layer="1"/>
-<wire x1="23.1775" y1="15.875" x2="24.4475" y2="15.875" width="0.4064" layer="1"/>
-<wire x1="24.4475" y1="15.875" x2="24.4475" y2="18.7325" width="0.4064" layer="1"/>
-<wire x1="24.4475" y1="18.7325" x2="25.885" y2="18.7325" width="0.4064" layer="1"/>
-<wire x1="25.885" y1="18.7325" x2="25.8875" y2="18.73" width="0.4064" layer="1"/>
+<wire x1="23.1775" y1="15.9775" x2="23.1775" y2="16.1925" width="0.4064" layer="1"/>
+<wire x1="23.1775" y1="16.1925" x2="24.62" y2="16.1925" width="0.4064" layer="1"/>
+<wire x1="24.62" y1="16.1925" x2="25.085" y2="15.7275" width="0.4064" layer="1"/>
 </signal>
 <signal name="N$3">
 <contactref element="Q1" pad="C"/>
 <contactref element="R4" pad="2"/>
-<wire x1="28.0875" y1="17.78" x2="29.21" y2="17.78" width="0.4064" layer="1"/>
-<wire x1="29.21" y1="17.78" x2="29.21" y2="15.025" width="0.4064" layer="1"/>
-<wire x1="29.21" y1="15.025" x2="29.1075" y2="14.9225" width="0.4064" layer="1"/>
+<wire x1="28.8925" y1="17.6775" x2="28.8925" y2="17.4625" width="0.4064" layer="1"/>
+<wire x1="28.8925" y1="17.4625" x2="26.035" y2="17.4625" width="0.4064" layer="1"/>
+<wire x1="26.035" y1="17.4625" x2="26.035" y2="17.9275" width="0.4064" layer="1"/>
 </signal>
 <signal name="CAP1">
@@
 <contactref element="R1" pad="2"/>
 <contactref element="IC3" pad="2"/>
-<wire x1="26.035" y1="12.125" x2="26.035" y2="13.97" width="0.4064" layer="1"/>
-<wire x1="26.035" y1="13.97" x2="25.4" y2="14.605" width="0.4064" layer="1"/>
 <wire x1="21.59" y1="10.375" x2="25.9325" y2="10.375" width="0.4064" layer="1"/>
 <wire x1="25.9325" y1="10.375" x2="26.035" y2="10.4775" width="0.4064" layer="1"/>
@@
 <via x="21.59" y="12.065" extent="1-16" drill="0.5"/>
 <wire x1="21.59" y1="12.065" x2="21.59" y2="10.375" width="0.4064" layer="1"/>
-<wire x1="25.4" y1="14.605" x2="25.4" y2="16.8275" width="0.4064" layer="1"/>
-<wire x1="25.4" y1="16.8275" x2="25.885" y2="16.8275" width="0.4064" layer="1"/>
-<wire x1="25.885" y1="16.8275" x2="25.8875" y2="16.83" width="0.4064" layer="1"/>
+<wire x1="26.035" y1="12.125" x2="26.035" y2="13.6525" width="0.4064" layer="1"/>
+<wire x1="26.035" y1="13.6525" x2="26.9875" y2="14.605" width="0.4064" layer="1"/>
+<wire x1="26.9875" y1="14.605" x2="26.9875" y2="15.725" width="0.4064" layer="1"/>
+<wire x1="26.9875" y1="15.725" x2="26.985" y2="15.7275" width="0.4064" layer="1"/>
 </signal>
 <signal name="CAP2">
 <contactref element="R4" pad="1"/>
 <contactref element="IC3" pad="1"/>
-<wire x1="27.305" y1="12.125" x2="27.305" y2="14.82" width="0.4064" layer="1"/>
-<wire x1="27.305" y1="14.82" x2="27.4075" y2="14.9225" width="0.4064" layer="1"/>
 <contactref element="CORE" pad="3"/>
 <wire x1="26.67" y1="3.4925" x2="24.13" y2="6.0325" width="0.4064" layer="16"/>
@@
 <wire x1="22.5425" y1="11.43" x2="22.5425" y2="14.2875" width="0.4064" layer="16"/>
 <wire x1="22.5425" y1="14.2875" x2="22.86" y2="14.605" width="0.4064" layer="16"/>
-<wire x1="22.86" y1="14.605" x2="25.7175" y2="14.605" width="0.4064" layer="16"/>
-<wire x1="25.7175" y1="14.605" x2="26.3525" y2="15.24" width="0.4064" layer="16"/>
-<via x="26.3525" y="15.24" extent="1-16" drill="0.5"/>
-<wire x1="26.3525" y1="15.24" x2="27.09" y2="15.24" width="0.4064" layer="1"/>
-<wire x1="27.09" y1="15.24" x2="27.4075" y2="14.9225" width="0.4064" layer="1"/>
+<wire x1="22.86" y1="14.605" x2="28.8925" y2="14.605" width="0.4064" layer="16"/>
+<via x="28.8925" y="14.605" extent="1-16" drill="0.5"/>
+<wire x1="28.8925" y1="14.605" x2="28.8925" y2="15.9775" width="0.4064" layer="1"/>
+<wire x1="27.305" y1="12.125" x2="27.305" y2="13.0175" width="0.4064" layer="1"/>
+<wire x1="27.305" y1="13.0175" x2="28.8925" y2="14.605" width="0.4064" layer="1"/>
 </signal>
 <signal name="N$4">

Commit message: Cleanup
Routing:
- net DGND: track 43.9 -> 45.6 mm
Other:
- board size 45.7 x 19.7 mm -> 45.7 x 19 mm
Changed lines of the file:
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@@
 <plain>
 <wire x1="0" y1="0" x2="45.7" y2="0" width="0" layer="20"/>
-<wire x1="45.7" y1="0" x2="45.7" y2="19.6725" width="0" layer="20"/>
-<wire x1="45.7" y1="19.6725" x2="0" y2="19.6725" width="0" layer="20"/>
-<wire x1="0" y1="19.6725" x2="0" y2="0" width="0" layer="20"/>
+<wire x1="45.7" y1="0" x2="45.7" y2="19.0375" width="0" layer="20"/>
+<wire x1="45.7" y1="19.0375" x2="0" y2="19.0375" width="0" layer="20"/>
+<wire x1="0" y1="19.0375" x2="0" y2="0" width="0" layer="20"/>
 </plain>
 <attributes>
@@
 <wire x1="14.9225" y1="6.985" x2="13.7125" y2="6.985" width="0.4064" layer="1"/>
 <wire x1="13.7125" y1="6.985" x2="13.6525" y2="6.925" width="0.4064" layer="1"/>
-<wire x1="16.51" y1="17.6775" x2="16.51" y2="18.7325" width="0.4064" layer="1"/>
-<via x="16.51" y="18.7325" extent="1-16" drill="0.5"/>
-<wire x1="16.51" y1="18.7325" x2="17.4625" y2="18.7325" width="0.4064" layer="16"/>
-<wire x1="17.4625" y1="18.7325" x2="17.4625" y2="5.08" width="0.4064" layer="16"/>
+<wire x1="16.51" y1="17.6775" x2="16.51" y2="17.4625" width="0.4064" layer="1"/>
+<wire x1="16.51" y1="17.4625" x2="15.24" y2="17.4625" width="0.4064" layer="1"/>
+<wire x1="15.24" y1="17.4625" x2="15.24" y2="18.0975" width="0.4064" layer="1"/>
+<via x="15.24" y="18.0975" extent="1-16" drill="0.5"/>
+<wire x1="15.24" y1="18.0975" x2="17.4625" y2="18.0975" width="0.4064" layer="16"/>
+<wire x1="17.4625" y1="18.0975" x2="17.4625" y2="5.08" width="0.4064" layer="16"/>
 <contactref element="DPWR" pad="2"/>
 <wire x1="14.9225" y1="6.985" x2="18.415" y2="3.4925" width="0.4064" layer="1"/>
