File: DCO/DCO core 1.0.sch (EAGLE design)
At the start: 54 parts, among them IC1 PIC16F18325SL, IC2 MAX5216, IC3 TL074D, IC5 4013D, IC8 TL074D, Q1 MMBT3906, Q3 MMBT3906, Q4 MMBT3906

Commit message: Finished layout of DCO core v1.0
Parts:
- removed C10, C11, C12, C4, C8, C9: 100nF, resistor:C-EUC0805
- removed D1, D2, D3, D4: (no value), diode:DIODE-SOD80C
- removed IC3, IC8: TL074D, linear:TL074D
- removed IC5: 4013D, joakim:4013D
- removed OUT: (no value), joakim:MA04-1J
- removed PGM: (no value), joakim:MA05-1J
- removed Q1, Q3, Q4: MMBT3906, transistor-pnp:MMBT3906LT1SMD
- removed R10: 22k, resistor:R-EU_R0805
- removed R11, R20: 68k, resistor:R-EU_R0805
- removed R12: 56k, resistor:R-EU_R0805
- removed R13, R14, R8: (no value), resistor:R-EU_R0805
- removed R15, R16, R17, R9: 100k, resistor:R-EU_R0805
- removed R18: 50k, resistor:R-EU_R0805
- removed R19: 200k, resistor:R-EU_R0805
- removed R21: 330k, resistor:R-EU_R0805
- removed SV3: (no value), joakim:MA01-1J
- added IC4: TL072D, joakim:TL072D
- added T1: (no value), transistor:MMBT3904LT1-NPN-SOT23-BEC
- C1: value 270pF -> 100nF
- R1: value 100k -> 56k
- R3: value 10k -> 100k
- R5: value 68k -> 100k
- R6: value 330k -> 100k
- R7: value (none) -> 68k
Connections:
- removed net +15V1: C4.1
- removed net +15V2: C9.1
- removed net -15V1: C8.2
- removed net -15V2: C10.2
- removed net CAP2: CORE.3, IC8A.-IN, IC8B.OUT, IC8D.+IN, R15.1, R17.1, R4.1
- removed net N$11: Q3.B, R5.2, R6.2
- removed net N$12: D1.C, IC3A.OUT, Q3.C, R7.2
- removed net N$13: IC8A.OUT, R9.1
- removed net N$14: Q4.B, R10.2, R9.2
- removed net N$15: IC3A.-IN, R7.1, R8.2
- removed net N$16: D2.C, IC3B.OUT, Q4.C, R13.2
- removed net N$17: D1.A, R11.1
- removed net N$18: D2.A, R12.1
- removed net N$19: D3.C, IC3D.-IN, R15.2, R16.1
- removed net N$20: IC3B.-IN, R13.1, R14.2
- removed net N$23: D3.A, D4.C, IC3D.OUT
- removed net N$24: D4.A, R16.2, R18.2
- removed net N$3: Q1.C, R4.2
- removed net N$5: PGM.1
- removed net N$6: PGM.2
- removed net N$7: PGM.3
- removed net N$8: PGM.4
- removed net N$9: PGM.5
- removed net PULSE_CV: R14.1
- removed net PULSE_OUT: OUT.3, R12.2
- removed net PWM_CV: IC8A.+IN, SV3.1
- removed net SUB_1OCT: IC5A.!Q, IC5A.D, IC5B.CLK, R5.1
- removed net SUB_2OCT: IC5B.!Q, IC5B.D, R20.1
- removed net SUB_OSC_CV: R8.1
- removed net SUB_OSC_OUT: OUT.4, R11.2
- removed net SYNC_POLARITY: IC1.VPP/MCLR/RA3, SYNC.1
- removed net TRI_OUT: C12.2, IC3C.OUT, R19.2
- removed net TRI_SYM: C12.1, IC3C.-IN, R17.2, R18.1, R19.1
- new net CALIBRATE: IC1.RC3, R6.1, R7.2
- net +15V: now also APWR.1, IC4P.V+; no longer APWR.3, IC3P.V+, IC8P.V+
- net +5V: now also C1.2; no longer C11.1, IC5P.VDD
- net -15V: now also APWR.3, IC4P.V-; no longer APWR.1, IC3P.V-, IC8P.V-
- net AGND: now also IC4A.+IN, IC4B.+IN, R7.1; no longer C10.1, C4.2, C8.1, C9.2, IC3A.+IN, IC3B.+IN, IC3C.+IN, IC3D.+IN, IC8B.+IN, Q3.E, Q4.E, R10.1, R3.1
- net CAP1: now also IC4A.-IN, T1.E; no longer IC8B.-IN, Q1.E
- net CHARGE_VOLTAGE: now also R5.1; no longer IC8C.+IN
- net CTRL_SPI_OUT: now also SYNC.2; no longer COM.4
- net DAC_SPI: now also IC1.SDI1/RC1; no longer IC1.RC2
- net DATA_READY: now also IC1.VPP/MCLR/RA3; no longer IC1.RA2
- net DGND: now also C1.1; no longer C11.2, IC5A.R, IC5A.S, IC5B.R, IC5B.S, IC5P.VSS, R21.1, R6.1
- net N$1: now also R4.2, T1.C; no longer R20.2, R21.2
- net N$10: now also IC4B.OUT, R3.2; no longer IC8C.-IN, IC8C.OUT
- net N$2: now also T1.B; no longer Q1.B
- net N$4: now also IC4B.-IN, R3.1, R5.2; no longer C1.2, R2.2, R3.2
- net SAW_OUT: now also CORE.3, IC4A.OUT, R4.1, R6.2; no longer IC8D.-IN, IC8D.OUT, OUT.2
- net SYNC: now also IC1.RA2, SYNC.1; no longer IC1.RC3, SYNC.2
- net TIMER_OUT: now also COM.4, IC1.RC2, R2.2; no longer C1.1, IC1.SDI1/RC1, IC5A.CLK, OUT.1
Other:
- note removed: "TODO: - Out - Sub osc - Saw buffer - Pwm CV - Pulse out"
- note removed: "TODO: Check resistor values"
- note removed: "TODO: Gjør hull mindre"
- note removed: "TODO: Replace with VCA"
- note removed: "TODO: Test with/without cap (104) in feedback loop"
- note removed: "TODO: This is an ideal diode. It lets the signal pass (inverted) if the input is positive. It will not work with a saw wave that is not centered. Perhaps it is possible to add a voltage at the positive pole?"
- moved on the sheet: APWR, C1, COM, CORE, DPWR, R1, R2, R3, R4, R5, R6, R7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

Commit message: Larger pin pads
Parts:
- APWR, CORE: device joakim:MA03-1J -> joakim:MA03-1JP
- COM: device joakim:MA04-1J -> joakim:MA04-1JP
- DPWR, SYNC: value MA02-1J -> MA02-1JP; device joakim:MA02-1J -> joakim:MA02-1JP
Changed lines of the file:
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@@
 <part name="SUPPLY14" library="supply2" deviceset="DGND" device=""/>
 <part name="SUPPLY15" library="supply2" deviceset="AGND" device=""/>
-<part name="COM" library="joakim" deviceset="MA04-1J" device=""/>
-<part name="CORE" library="joakim" deviceset="MA03-1J" device=""/>
-<part name="APWR" library="joakim" deviceset="MA03-1J" device=""/>
-<part name="DPWR" library="joakim" deviceset="MA02-1J" device="" value=""/>
-<part name="SYNC" library="joakim" deviceset="MA02-1J" device="" value=""/>
+<part name="COM" library="joakim" deviceset="MA04-1J" device="P"/>
+<part name="CORE" library="joakim" deviceset="MA03-1J" device="P"/>
+<part name="APWR" library="joakim" deviceset="MA03-1J" device="P"/>
+<part name="DPWR" library="joakim" deviceset="MA02-1J" device="P" value="MA02-1JP"/>
+<part name="SYNC" library="joakim" deviceset="MA02-1J" device="P" value="MA02-1JP"/>
 <part name="T1" library="transistor" deviceset="*-NPN-" device="SOT23-BEC" technology="MMBT3904LT1"/>
 <part name="R3" library="resistor" deviceset="R-EU_" device="R0805" value="100k"/>
@@
 <instance part="CORE" gate="G$1" x="147.32" y="-5.08" rot="R180"/>
 <instance part="APWR" gate="G$1" x="147.32" y="50.8" rot="R180"/>
-<instance part="DPWR" gate="G$1" x="147.32" y="30.48" rot="R180"/>
-<instance part="SYNC" gate="G$1" x="147.32" y="-20.32" rot="R180"/>
+<instance part="DPWR" gate="G$1" x="147.32" y="30.48" smashed="yes" rot="R180">
+<attribute name="NAME" x="148.59" y="27.178" size="1.778" layer="95" rot="R180"/>
+</instance>
+<instance part="SYNC" gate="G$1" x="147.32" y="-20.32" smashed="yes" rot="R180">
+<attribute name="NAME" x="148.59" y="-23.622" size="1.778" layer="95" rot="R180"/>
+</instance>
 <instance part="T1" gate="G$1" x="45.72" y="-12.7" rot="R270"/>
 <instance part="R3" gate="G$1" x="7.62" y="-22.86" smashed="yes">
