File: Xonik Waveformer/Xonik Waveformer v1.0.sch (EAGLE design)
At the start: 84 parts, among them IC1 TL074D, IC2 TL074D, IC3 TL074D, IC4 4013D, IC5 TL072D

Commit message: Working with board layout
Parts:
- removed R21, R31, R32, R33, R34, R42, R43, R57: 1k, resistor:R-EU_R0805
- removed R51, R52, R54: 100k, resistor:R-TRIMM3296W
- removed R53: 50k, resistor:R-TRIMM3296W
- added +15V, +5V, -15V, CENTER, DCO_IN, DCO_TIMER, GND, INV_SAW, PULSE, PULSE_AMP_CV, PW_CV, SAW, SINE, ST1, ST2, ST3, ST4, SUB_SAW_1, SUB_SAW_2, SUB_SQR2, SUB_SQR_1, SYMMETRY, TRIANGLE: (no value), joakim:MA01-1J
- C5, C6: value (none) -> 100nF
- D1, D2, D3, D4: value (none) -> 1N41480805; device diode:DIODE-D-5 -> joakim:1N41480805
- IC4: value 4013D -> TL072D; device joakim:4013D -> joakim:TL072D
- IC5: value TL072D -> 4013D; device joakim:TL072D -> joakim:4013D
- R9: value 1k -> 330k
- T1: value (none) -> 2n3904
Connections:
- removed net N$25: IC3D.OUT, R38.2, R52.A, R52.S
- removed net N$42: C13.2, C9.1
- removed net N$43: C10.1, C14.2
- removed net N$44: C11.1, C15.2
- new net N$41: IC3C.OUT, R38.2, ST2.1
- net +15V: now also +15V.1, C10.2, C11.2, C9.2, IC4P.V+
- net +5V: now also +5V.1, IC5P.VDD; no longer IC4P.VDD
- net -15V: now also -15V.1, C13.1, C14.1, C15.1, IC4P.V-; no longer R54.A, R54.S
- net AMP_CV: now also PULSE_AMP_CV.1
- net DCO_IN: now also DCO_IN.1
- net GND: now also C10.1, C11.1, C13.2, C14.2, C15.2, C9.1, GND.1, IC1C.+IN, IC4A.+IN, IC4B.+IN, IC5A.R, IC5A.S, IC5B.R, IC5B.S, IC5P.VSS; no longer IC1B.+IN, IC2C.+IN, IC4A.R, IC4A.S, IC4B.R, IC4B.S, IC4P.VSS, IC5A.+IN
- net N$10: now also CENTER.1, IC1A.-IN; no longer IC1B.-IN, R54.E
- net N$11: now also IC1C.-IN; no longer IC1A.-IN
- net N$12: now also IC1C.OUT; no longer IC1A.OUT
- net N$14: now also IC2D.-IN; no longer IC5A.-IN
- net N$15: now also IC2A.-IN; no longer IC2D.-IN
- net N$16: now also IC2A.OUT, SAW.1; no longer IC2D.OUT, R32.1
- net N$17: now also IC4B.OUT, SUB_SQR_1.1; no longer IC2C.OUT, R33.1
- net N$18: now also IC4A.OUT, SUB_SQR2.1; no longer IC2A.OUT, R34.1
- net N$19: now also IC4B.-IN; no longer IC2C.-IN
- net N$20: now also ST4.1; no longer R51.A, R51.S
- net N$22: now also IC4A.-IN; no longer IC2A.-IN
- net N$24: now also IC3C.-IN, ST1.1; no longer IC3D.-IN, R52.E
- net N$26: now also IC3D.-IN; no longer IC3C.-IN
- net N$27: now also IC3D.OUT, SUB_SAW_1.1; no longer IC3C.OUT, R42.1
- net N$28: now also ST3.1; no longer R51.E
- net N$3: now also R9.1
- net N$30: now also SUB_SAW_2.1; no longer R43.1
- net N$31: now also IC5A.!Q, IC5A.D; no longer IC4A.!Q, IC4A.D
- net N$32: now also IC5A.Q, IC5B.CLK; no longer IC4A.Q, IC4B.CLK
- net N$34: now also IC5B.!Q, IC5B.D; no longer IC4B.!Q, IC4B.D
- net N$35: now also IC5B.Q; no longer IC4B.Q
- net N$36: now also IC2C.-IN; no longer IC5B.-IN
- net N$37: now also SYMMETRY.1; no longer R53.S
- net N$38: now also IC2D.OUT, TRIANGLE.1; no longer IC5A.OUT, R57.1
- net N$39: now also IC2C.+IN; no longer IC5B.+IN
- net N$40: now also IC2C.OUT, SINE.1; no longer IC5B.OUT, R21.2
- net N$6: now also IC1B.-IN; no longer IC1C.-IN
- net N$7: now also IC1B.OUT, PULSE.1; no longer IC1C.OUT, R9.1
- net N$8: now also IC1B.+IN; no longer IC1C.+IN
- net N$9: now also IC1A.OUT, INV_SAW.1; no longer IC1B.OUT, R31.1
- net PW_CV: now also PW_CV.1
- net SQR: now also DCO_TIMER.1, IC5A.CLK; no longer IC4A.CLK
Other:
- note added: "All caps 100nF"
- note added: "Ext 100k pot"
- note added: "Ext 100k pot to -15V"
- note added: "Ext pot GND to +15V"
- note removed: "switch diodes"
- moved on the sheet: IC1A, IC1B, IC1C, IC2A, IC2C, IC2D, IC3C, IC3D, R9

Commit message: Still doing layout
Parts:
- removed TP1: TPPAD1-13, testpad:TPPAD1-13
Connections:
- net N$9: no longer TP1.TP
Changed lines of the file:
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@@
 <part name="T1" library="transistor-neu-to92" deviceset="*-NPN-" device="SOT23-BEC" technology="MMBT3904LT1" value="2n3904"/>
 <part name="GND2" library="supply1" deviceset="GND" device=""/>
-<part name="TP1" library="testpad" deviceset="TP" device="PAD1-13"/>
 <part name="GND3" library="supply1" deviceset="GND" device=""/>
 <part name="GND4" library="supply1" deviceset="GND" device=""/>
@@
 </instance>
 <instance part="GND2" gate="1" x="38.1" y="76.2"/>
-<instance part="TP1" gate="G$1" x="-2.54" y="60.96" rot="R90"/>
 <instance part="GND3" gate="1" x="-25.4" y="40.64"/>
 <instance part="GND4" gate="1" x="12.7" y="43.18"/>
@@
 <pinref part="IC1" gate="D" pin="-IN"/>
 <wire x1="2.54" y1="86.36" x2="0" y2="86.36" width="0.1524" layer="91"/>
-<wire x1="0" y1="86.36" x2="0" y2="60.96" width="0.1524" layer="91"/>
-<pinref part="TP1" gate="G$1" pin="TP"/>
-<wire x1="0" y1="60.96" x2="0" y2="50.8" width="0.1524" layer="91"/>
-<junction x="0" y="60.96"/>
+<wire x1="0" y1="86.36" x2="0" y2="50.8" width="0.1524" layer="91"/>
 <pinref part="IC1" gate="A" pin="OUT"/>
 <wire x1="0" y1="50.8" x2="0" y2="45.72" width="0.1524" layer="91"/>

Commit message: Routing complete except for bypass caps
Parts:
- added GND27: (no value), joakim:MA01-1J
Connections:
- removed net N$8: IC1B.+IN, R6.2
- net GND: now also GND27.1, R6.2
- net N$5: now also IC1B.+IN
Changed lines of the file:
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@@
 <part name="ST3" library="joakim" deviceset="MA01-1J" device=""/>
 <part name="ST4" library="joakim" deviceset="MA01-1J" device=""/>
+<part name="GND26" library="supply1" deviceset="GND" device=""/>
+<part name="GND27" library="joakim" deviceset="MA01-1J" device=""/>
 </parts>
 <sheets>
 <sheet>
 <plain>
-<text x="12.7" y="73.66" size="1.778" layer="91">NB: 330k?</text>
+<text x="-7.62" y="116.84" size="1.778" layer="91">NB: 330k?</text>
 <text x="129.54" y="22.86" size="1.778" layer="97">All caps 100nF</text>
 <text x="-48.26" y="27.94" size="1.778" layer="97">Ext 100k pot to -15V</text>
@@
 <attribute name="NAME" x="36.83" y="-89.662" size="1.778" layer="95" rot="R180"/>
 </instance>
+<instance part="GND26" gate="1" x="60.96" y="91.44"/>
+<instance part="GND27" gate="G$1" x="121.92" y="33.02"/>
 </instances>
 <busses>
@@
 <pinref part="C15" gate="G$1" pin="2"/>
 <junction x="149.86" y="40.64"/>
+<pinref part="GND27" gate="G$1" pin="1"/>
+<wire x1="129.54" y1="33.02" x2="129.54" y2="40.64" width="0.1524" layer="91"/>
+<junction x="129.54" y="40.64"/>
+</segment>
+<segment>
+<pinref part="R6" gate="G$1" pin="2"/>
+<pinref part="GND26" gate="1" pin="GND"/>
 </segment>
 </net>
@@
 <pinref part="R6" gate="G$1" pin="1"/>
 <wire x1="55.88" y1="104.14" x2="60.96" y2="104.14" width="0.1524" layer="91"/>
+<wire x1="60.96" y1="104.14" x2="66.04" y2="104.14" width="0.1524" layer="91"/>
+<pinref part="IC1" gate="B" pin="+IN"/>
+<wire x1="66.04" y1="83.82" x2="71.12" y2="83.82" width="0.1524" layer="91"/>
+<wire x1="66.04" y1="104.14" x2="66.04" y2="83.82" width="0.1524" layer="91"/>
 </segment>
 </net>
@@
 </segment>
 </net>
-<net name="N$8" class="0">
-<segment>
-<pinref part="R6" gate="G$1" pin="2"/>
-<wire x1="60.96" y1="93.98" x2="60.96" y2="83.82" width="0.1524" layer="91"/>
-<pinref part="IC1" gate="B" pin="+IN"/>
-<wire x1="60.96" y1="83.82" x2="71.12" y2="83.82" width="0.1524" layer="91"/>
-</segment>
-</net>

Commit message: Finished tracing, working on labels
Parts:
- C10, C11, C12, C13, C14, C15, C8, C9: device resistor:C-EUC0805 -> resistor:C-EUC0603K
- renumbered R1 to 1, R10 to 10, R11 to 11, R12 to 12, R13 to 13, R14 to 14, R15 to 15, R16 to 16, R17 to 17, R18 to 18, R19 to 19, R2 to 2, R20 to 20, R22 to 22, R23 to 23, R24 to 24, R25 to 25, R26 to 26, R27 to 27, R28 to 28, R29 to 29, R3 to 3, R30 to 30, R35 to 35, R36 to 36, R37 to 37, R38 to 38, R39 to 39, R4 to 4, R40 to 40, R41 to 41, R44 to 44, R45 to 45, R46 to 46, R47 to 47, R48 to 48, R49 to 49, R5 to 5, R50 to 50, R55 to 55, R56 to 56, R6 to 6, R7 to 7, R8 to 8, R9 to 9
Connections:
- net GND: now also 9.2

Commit message: Trace and text complete, gp and logo missing
Parts:
- removed SUB_SQR2: (no value), joakim:MA01-1J
- added SUB_SQR_2: (no value), joakim:MA01-1JP
- +15V, +5V, -15V, CENTER, DCO_IN, DCO_TIMER, GND, GND27, INV_SAW, PULSE, PULSE_AMP_CV, PW_CV, SAW, SINE, ST1, ST2, ST3, ST4, SUB_SAW_1, SUB_SAW_2, SUB_SQR_1, SYMMETRY, TRIANGLE: device joakim:MA01-1J -> joakim:MA01-1JP
- C16: device resistor:C-EUC0805 -> resistor:C-EUC0603K
- C8: device resistor:C-EUC0603K -> resistor:C-EUC0805
Connections:
- net +15V: now also C16.2; no longer C8.2
- net +5V: now also C8.2; no longer C16.2
- net N$18: now also SUB_SQR_2.1; no longer SUB_SQR2.1
Other:
- moved on the sheet: C16, C8
Changed lines of the file:
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@@
 <part name="D3" library="joakim" deviceset="1N4148" device="0805"/>
 <part name="D4" library="joakim" deviceset="1N4148" device="0805"/>
-<part name="C8" library="resistor" deviceset="C-EU" device="C0603K" value="100nF"/>
+<part name="C16" library="resistor" deviceset="C-EU" device="C0603K" value="100nF"/>
 <part name="C9" library="resistor" deviceset="C-EU" device="C0603K" value="100nF"/>
 <part name="C10" library="resistor" deviceset="C-EU" device="C0603K" value="100nF"/>
@@
 <part name="SUPPLY6" library="supply2" deviceset="+15V" device=""/>
 <part name="SUPPLY7" library="supply2" deviceset="-15V" device=""/>
-<part name="C16" library="resistor" deviceset="C-EU" device="C0805" value="100nF"/>
-<part name="PULSE" library="joakim" deviceset="MA01-1J" device=""/>
-<part name="SINE" library="joakim" deviceset="MA01-1J" device=""/>
-<part name="TRIANGLE" library="joakim" deviceset="MA01-1J" device=""/>
-<part name="INV_SAW" library="joakim" deviceset="MA01-1J" device=""/>
-<part name="SAW" library="joakim" deviceset="MA01-1J" device=""/>
-<part name="SUB_SQR_1" library="joakim" deviceset="MA01-1J" device=""/>
-<part name="SUB_SAW_1" library="joakim" deviceset="MA01-1J" device=""/>
-<part name="SUB_SQR2" library="joakim" deviceset="MA01-1J" device=""/>
-<part name="SUB_SAW_2" library="joakim" deviceset="MA01-1J" device=""/>
-<part name="PULSE_AMP_CV" library="joakim" deviceset="MA01-1J" device=""/>
-<part name="PW_CV" library="joakim" deviceset="MA01-1J" device=""/>
-<part name="DCO_IN" library="joakim" deviceset="MA01-1J" device=""/>
-<part name="+15V" library="joakim" deviceset="MA01-1J" device=""/>
-<part name="GND" library="joakim" deviceset="MA01-1J" device=""/>
-<part name="-15V" library="joakim" deviceset="MA01-1J" device=""/>
-<part name="+5V" library="joakim" deviceset="MA01-1J" device=""/>
-<part name="DCO_TIMER" library="joakim" deviceset="MA01-1J" device=""/>
+<part name="C8" library="resistor" deviceset="C-EU" device="C0805" value="100nF"/>
+<part name="PULSE" library="joakim" deviceset="MA01-1J" device="P"/>
+<part name="SINE" library="joakim" deviceset="MA01-1J" device="P"/>
+<part name="TRIANGLE" library="joakim" deviceset="MA01-1J" device="P"/>
+<part name="INV_SAW" library="joakim" deviceset="MA01-1J" device="P"/>
+<part name="SAW" library="joakim" deviceset="MA01-1J" device="P"/>
+<part name="SUB_SQR_1" library="joakim" deviceset="MA01-1J" device="P"/>
+<part name="SUB_SAW_1" library="joakim" deviceset="MA01-1J" device="P"/>
+<part name="SUB_SQR_2" library="joakim" deviceset="MA01-1J" device="P"/>
+<part name="SUB_SAW_2" library="joakim" deviceset="MA01-1J" device="P"/>
+<part name="PULSE_AMP_CV" library="joakim" deviceset="MA01-1J" device="P"/>
+<part name="PW_CV" library="joakim" deviceset="MA01-1J" device="P"/>
+<part name="DCO_IN" library="joakim" deviceset="MA01-1J" device="P"/>
+<part name="+15V" library="joakim" deviceset="MA01-1J" device="P"/>
+<part name="GND" library="joakim" deviceset="MA01-1J" device="P"/>
+<part name="-15V" library="joakim" deviceset="MA01-1J" device="P"/>
+<part name="+5V" library="joakim" deviceset="MA01-1J" device="P"/>
+<part name="DCO_TIMER" library="joakim" deviceset="MA01-1J" device="P"/>
 <part name="9" library="resistor" deviceset="R-EU_" device="R0805" value="330k"/>
-<part name="CENTER" library="joakim" deviceset="MA01-1J" device=""/>
-<part name="SYMMETRY" library="joakim" deviceset="MA01-1J" device=""/>
-<part name="ST1" library="joakim" deviceset="MA01-1J" device=""/>
-<part name="ST2" library="joakim" deviceset="MA01-1J" device=""/>
-<part name="ST3" library="joakim" deviceset="MA01-1J" device=""/>
-<part name="ST4" library="joakim" deviceset="MA01-1J" device=""/>
+<part name="CENTER" library="joakim" deviceset="MA01-1J" device="P"/>
+<part name="SYMMETRY" library="joakim" deviceset="MA01-1J" device="P"/>
+<part name="ST1" library="joakim" deviceset="MA01-1J" device="P"/>
+<part name="ST2" library="joakim" deviceset="MA01-1J" device="P"/>
+<part name="ST3" library="joakim" deviceset="MA01-1J" device="P"/>
+<part name="ST4" library="joakim" deviceset="MA01-1J" device="P"/>
 <part name="GND26" library="supply1" deviceset="GND" device=""/>
-<part name="GND27" library="joakim" deviceset="MA01-1J" device=""/>
+<part name="GND27" library="joakim" deviceset="MA01-1J" device="P"/>
 <part name="GND28" library="supply1" deviceset="GND" device=""/>
 </parts>
@@
 <attribute name="NAME" x="83.82" y="56.3626" size="1.778" layer="95"/>
 </instance>
-<instance part="C8" gate="G$1" x="134.62" y="43.18" smashed="yes" rot="R180">
+<instance part="C16" gate="G$1" x="134.62" y="43.18" smashed="yes" rot="R180">
 <attribute name="NAME" x="132.461" y="51.816" size="1.778" layer="95" rot="R270"/>
 </instance>
@@
 <instance part="SUPPLY6" gate="+15V" x="154.94" y="50.8"/>
 <instance part="SUPPLY7" gate="G$1" x="154.94" y="30.48"/>
-<instance part="C16" gate="G$1" x="160.02" y="73.66" smashed="yes" rot="R180">
+<instance part="C8" gate="G$1" x="160.02" y="73.66" smashed="yes" rot="R180">
 <attribute name="NAME" x="157.861" y="72.136" size="1.778" layer="95" rot="R270"/>
 <attribute name="VALUE" x="162.179" y="65.024" size="1.778" layer="96" rot="R90"/>
@@
 <instance part="SUB_SQR_1" gate="G$1" x="99.06" y="-20.32" rot="R180"/>
 <instance part="SUB_SAW_1" gate="G$1" x="99.06" y="-40.64" rot="R180"/>
-<instance part="SUB_SQR2" gate="G$1" x="99.06" y="-78.74" rot="R180"/>
+<instance part="SUB_SQR_2" gate="G$1" x="99.06" y="-78.74" rot="R180"/>
 <instance part="SUB_SAW_2" gate="G$1" x="99.06" y="-99.06" rot="R180"/>
 <instance part="PULSE_AMP_CV" gate="G$1" x="-35.56" y="104.14"/>
@@
 <pinref part="IC5" gate="P" pin="VSS"/>
 <pinref part="GND21" gate="1" pin="GND"/>
-<pinref part="C16" gate="G$1" pin="1"/>
+<pinref part="C8" gate="G$1" pin="1"/>
 <wire x1="160.02" y1="71.12" x2="160.02" y2="66.04" width="0.1524" layer="91"/>
 <wire x1="160.02" y1="66.04" x2="152.4" y2="66.04" width="0.1524" layer="91"/>
@@
 </segment>
 <segment>
-<pinref part="C8" gate="G$1" pin="1"/>
+<pinref part="C16" gate="G$1" pin="1"/>
 <pinref part="C12" gate="G$1" pin="2"/>
 <wire x1="134.62" y1="40.64" x2="139.7" y2="40.64" width="0.1524" layer="91"/>
@@
 <wire x1="33.02" y1="-60.96" x2="33.02" y2="-68.58" width="0.1524" layer="91"/>
 <junction x="33.02" y="-68.58"/>
-<pinref part="SUB_SQR2" gate="G$1" pin="1"/>
+<pinref part="SUB_SQR_2" gate="G$1" pin="1"/>
 </segment>
 </net>
@@
 <pinref part="IC5" gate="P" pin="VDD"/>
 <pinref part="SUPPLY3" gate="+5V" pin="+5V"/>
-<pinref part="C16" gate="G$1" pin="2"/>
+<pinref part="C8" gate="G$1" pin="2"/>
 <wire x1="160.02" y1="78.74" x2="160.02" y2="81.28" width="0.1524" layer="91"/>
 <wire x1="160.02" y1="81.28" x2="152.4" y2="81.28" width="0.1524" layer="91"/>
@@
 </segment>
 <segment>
-<pinref part="C8" gate="G$1" pin="2"/>
+<pinref part="C16" gate="G$1" pin="2"/>
 <wire x1="134.62" y1="48.26" x2="139.7" y2="48.26" width="0.1524" layer="91"/>
 <pinref part="SUPPLY6" gate="+15V" pin="+15V"/>
