File: Xonik Waveformer/Xonik Waveshaper v1.0-take 2.brd (EAGLE design)
At the start: 63.5 x 28.3 mm, 94 parts, among them IC1 TL074D, IC2 TL074D, IC3 TL074D, IC4 TL072D, IC5 4013D, T1 2n3904

Commit message: Probably final version before adding gp and stuff
Parts:
- moved D1 2.54 mm to (17.1, 23.8)
- moved D2 2.54 mm to (14.6, 23.8), turned to 90 degrees
Routing:
- net N$13: track 13.5 -> 7.02 mm
- net GND: track 289.6 -> 293.2 mm
- net -2.5V: track 71.0 -> 72.2 mm
- net N$12: track 11.8 -> 10.5 mm
- net N$11: track 11.5 -> 12.6 mm
