File: Xonik Waveformer/Xonik Waveshaper v1.0 w gp.brd (EAGLE design)
At the start: 63.5 x 28.3 mm, 94 parts, among them IC1 TL074D, IC2 TL074D, IC3 TL074D, IC4 TL072D, IC5 4013D, T1 2n3904

Commit message: Added logo, only panelizing is missing
Parts:
- turned T1 to 180 degrees
Routing:
- net N$4: track 25.8 -> 23.6 mm
- net N$3: track 12.5 -> 10.8 mm
- net GND: track 290.1 -> 289.3 mm
Other:
- board text added: "1"
- board text added: "10"
- board text added: "11"
- board text added: "12"
- board text added: "13"
- board text added: "14"
- board text added: "15"
- board text added: "16"
- board text added: "17"
- board text added: "18"
- board text added: "19"
- board text added: "2"
- board text added: "20"
- board text added: "22"
- board text added: "23"
- board text added: "24"
- board text added: "25"
- board text added: "26"
- board text added: "27"
- board text added: "28"
- board text added: "29"
- board text added: "3"
- board text added: "30"
- board text added: "35"
- board text added: "36"
- board text added: "37"
- board text added: "38"
- board text added: "39"
- board text added: "4"
- board text added: "40"
- board text added: "41"
- board text added: "44"
- board text added: "45"
- board text added: "46"
- board text added: "47"
- board text added: "48"
- board text added: "49"
- board text added: "4V&B"
- board text added: "5"
- board text added: "50"
- board text added: "55"
- board text added: "56"
- board text added: "6"
- board text added: "7"
- board text added: "8"
- board text added: "C1"
- board text added: "C2"
- board text added: "C3"
- board text added: "C4"
- board text added: "C5"
- board text added: "C6"
- board text added: "C7"
- board text added: "C8"
- board text added: "D1"
- board text added: "D2"
- board text added: "D3"
- board text added: "D4"
- board text added: "IC1"
- board text added: "IC2"
- board text added: "IC3"
- board text added: "IC4"
- board text added: "IC5"
- board text added: "T1"
- board text added: "XWS"
- board text added: "v1.0"
